Commit message: feat(*): 机械臂更新urdf文件

File: app/src/main/assets/urdf/URDF_armv001_a3tip.urdf (robot description, URDF)
Before this commit: robot URDF_armv001_a3tip, 7 links, 6 joints
Links:
- link base_link: geometry collision mesh filename=meshes/base_link.STL; visual mesh filename=meshes/base_link.STL
- link fifth_Link: geometry collision mesh filename=meshes/fifth_Link.STL; collision mesh filename=meshes/jaw.stl
- link first_Link: geometry collision mesh filename=meshes/first_Link.STL; visual mesh filename=meshes/first_Link.STL
- link fourth_Link: geometry collision mesh filename=meshes/fourth_Link.STL; visual mesh filename=meshes/fourth_Link.STL
- link second_Link: geometry collision mesh filename=meshes/second_arm_asm.stl; visual mesh filename=meshes/second_arm_asm.stl
- link third_Link: geometry collision mesh filename=meshes/third_Link.STL; visual mesh filename=meshes/third_Link.STL
Joints:
- joint third_joint: origin xyz=0 0.165989898732231 0.257913780286487 rpy=0 0 0 -> xyz=0 0.141086 0.244377 rpy=0 0 0
